Commit message: URDF copy: ToF on top of the ZED, 20 deg down
zed_camera_link -> tof: xyz (0, 0, 0.041) = centred on top of the ZED 2i
(30 mm tall) plus ~11 mm to the TFmini Plus lens centre; pitch 20 deg down.

Co-Authored-By: Claude Opus 5.5 <noreply@anthropic.com>

File: orin_files/cac_rover_to_cpy.urdf (robot description, URDF)
Before this commit: robot cac_rover, 24 links, 23 joints
Joints:
- joint zed_to_tof: origin xyz=0.04 0.0 -0.02 rpy=0.0 0.3490658503988659 0.0 -> xyz=0.0 0.0 0.041 rpy=0.0 0.3490658503988659 0.0

Commit message: ToF tilt 33 deg (d ~ 1.2 m): URDF pitch and jump_threshold 0.09
At ~0.65 m height, 33 deg down gives a flat-ground reading of ~1.2 m,
~1.0 m ahead. A crater of depth D lengthens the reading by D/sin(33),
so jump_threshold 0.09 m keeps detecting ~5 cm deep craters.

Co-Authored-By: Claude Opus 5.5 <noreply@anthropic.com>

File: orin_files/cac_rover_to_cpy.urdf (robot description, URDF)
Before this commit: robot cac_rover, 24 links, 23 joints
Joints:
- joint zed_to_tof: origin xyz=0.0 0.0 0.041 rpy=0.0 0.3490658503988659 0.0 -> xyz=0.0 0.0 0.041 rpy=0.0 0.5759586531581288 0.0
